File: esp.kicad_sch (KiCad schematic)
At the start: 45 parts, among them J1 USB_C_Receptacle_USB2.0_14P, J2 Conn_01x06_Pin, SW1 RESET, SW2 BOOT, U1 ESP32-C3, U2 W25Q128JVP, U3 USBLC6-2P6, U4 MS5611-01BA, U5 SPX3819M5-L-3-3, U6 SHTC3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

Commit message: pushing before redoing everything
Parts:
- removed J2: Conn_01x06_Pin, Connector_PinHeader_2.54mm:PinHeader_2x03_P2.54mm_Vertical, symbol Connector:Conn_01x06_Pin
- added J2: Conn_01x04_Pin, Connector_PinHeader_2.54mm:PinHeader_1x04_P2.54mm_Vertical, symbol Connector:Conn_01x04_Pin
- AE1: footprint (none) -> RF_Antenna:Texas_SWRA117D_2.4GHz_Left
- C20, C21, C4, C5, C6, C8, C9: footprint Capacitor_SMD:C_0603_1608Metric -> Capacitor_SMD:C_0402_1005Metric
- L1, L2, L3: footprint Inductor_SMD:L_0805_2012Metric -> Inductor_SMD:L_0402_1005Metric
- R1, R2, R3, R4, R5, R6, R7, R8, R9: footprint Resistor_SMD:R_0603_1608Metric_Pad0.98x0.95mm_HandSolder -> Resistor_SMD:R_0402_1005Metric
- U2: footprint Package_SON:WSON-8-1EP_6x5mm_P1.27mm_EP3.4x4.3mm -> Package_SON:Winbond_USON-8-2EP_3x4mm_P0.8mm_EP0.2x0.8mm
Connections:
- net +3V3: now also J2.1 (Pin_1)
- net GND: now also U3.2 (GND), J2.4 (Pin_4)
- net MCS: now also U1.8 (GPIO3)
- net RXD: now also J2.2 (Pin_2)
- net TXD: now also J2.3 (Pin_3)
- net VBUS: now also U3.5 (VBUS)
- net DO-: now reaches J1.A7 (D-), J1.B7 (D-), U3.1 (I/O1)
- net DO+: now reaches J1.A6 (D+), J1.B6 (D+), U3.3 (I/O2)
Other:
- moved on the sheet: AE1, U3
