File: esp.kicad_pcb (KiCad board)
At the start: 2 copper layers, 41 parts, among them J1 USB_C_Receptacle_USB2.0_14P, J2 Conn_01x06_Pin, SW1 RESET, SW2 BOOT, U1 ESP32-C3, U2 W25Q128JVP, U3 USBLC6-2P6, U4 MS5611-01BA, U5 SPX3819M5-L-3-3, U6 SHTC3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

Commit message: pushing before redoing everything
Parts:
- added AE1: Antenna_Shield, RF_Antenna:Texas_SWRA117D_2.4GHz_Left, F.Cu at (165.8, 72.8)
- added C20: 3.3pF, Capacitor_SMD:C_0402_1005Metric, F.Cu at (168.2, 67.8)
- added C21: 3.3pF, Capacitor_SMD:C_0402_1005Metric, F.Cu at (168.2, 70.8)
- added L3: 2.2nH, Inductor_SMD:L_0402_1005Metric, F.Cu at (168.7, 69.3)
- C4, C5, C6, C8, C9: footprint Capacitor_SMD:C_0603_1608Metric -> Capacitor_SMD:C_0402_1005Metric
- J2: value Conn_01x06_Pin -> Conn_01x04_Pin; footprint Connector_PinHeader_2.54mm:PinHeader_2x03_P2.54mm_Vertical -> Connector_PinHeader_2.54mm:PinHeader_1x04_P2.54mm_Vertical
- L1, L2: footprint Inductor_SMD:L_0805_2012Metric -> Inductor_SMD:L_0402_1005Metric
- R1, R2, R3, R4, R5, R6, R7, R8, R9: footprint Resistor_SMD:R_0603_1608Metric_Pad0.98x0.95mm_HandSolder -> Resistor_SMD:R_0402_1005Metric
- U2: footprint Package_SON:WSON-8-1EP_6x5mm_P1.27mm_EP3.4x4.3mm -> Package_SON:Winbond_USON-8-2EP_3x4mm_P0.8mm_EP0.2x0.8mm
- moved L2 68.3 mm to (175.4, 49.2)
- moved J1 67.8 mm to (170.2, 41.4), turned to 180 degrees
- moved U5 64.3 mm to (175.2, 53.0), turned to -90 degrees
- moved U3 62.8 mm to (170.2, 50.4), turned to -90 degrees
- moved C14 62.6 mm to (172.6, 50.1), turned to -90 degrees
- moved R7 60.1 mm to (176.2, 44.8), turned to 90 degrees
- moved C15 59.4 mm to (175.2, 56.1), turned to 180 degrees
- moved U6 57.3 mm to (178.2, 59.1), turned to -90 degrees
- moved SW1 56.2 mm to (162.2, 40.8), turned to -90 degrees
- moved SW2 55.4 mm to (178.2, 40.8), turned to -90 degrees
- moved R6 55.4 mm to (168.4, 47.4), turned to -90 degrees
- moved C13 53.2 mm to (175.4, 47.4)
- moved R5 52.6 mm to (171.4, 47.4), turned to -90 degrees
- moved U4 51.5 mm to (178.1, 64.5)
- moved R8 50.4 mm to (178.0, 57.1), turned to 180 degrees
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Connections:
- net Net-(J1-D+-PadA6) renamed DO+
- net Net-(J1-D--PadA7) renamed DO-
- J2 pad 1: SDO -> +3V3
- J2 pad 2: SDI -> RXD
- J2 pad 3: SCLK -> TXD
- J2 pad 4: SCS -> GND
- U1 pad 1: unconnected-(U1-LNA_IN-Pad1) -> Net-(U1-LNA_IN)
- U1 pad 8: unconnected-(U1-GPIO3-Pad8) -> MCS
- U3 pad 2: unconnected-(U3-GND-Pad2) -> GND
- U3 pad 5: unconnected-(U3-VBUS-Pad5) -> VBUS
Routing:
- net GND: track 0.00 -> 40.0 mm, vias 0 -> 63
- net EN: track 0.00 -> 39.4 mm, vias 0 -> 2
- net BOOT: track 0.00 -> 32.7 mm, vias 0 -> 2
- net +3V3: track 0.00 -> 30.8 mm, vias 0 -> 10
- net VBUS: track 0.00 -> 18.1 mm
- net D+: track 0.00 -> 15.8 mm
- net D-: track 0.00 -> 15.0 mm
- net V_FILT: track 0.00 -> 13.3 mm
- net Net-(U1-U0RXD): track 0.00 -> 12.9 mm
- net Net-(U1-U0TXD): track 0.00 -> 11.2 mm, vias 0 -> 2
- net SDO: track 0.00 -> 9.39 mm
- net SCL: track 0.00 -> 9.37 mm
- net SCS: track 0.00 -> 7.78 mm, vias 0 -> 2
- net DO+: track 0.00 -> 7.35 mm
- net DO-: track 0.00 -> 7.35 mm
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- added copper zone on B.Cu, net +3V3
- added copper zone on F.Cu, net GND
- added copper zone on In1.Cu, net GND
- added copper zone on In2.Cu, net GND
Other:
- board outline added: 20 x 40.8 mm
- copper layers 2 -> 4

Commit message: pushing before redoing everything
Parts:
- moved SW1 30.1 mm to (151.9, 69.0), turned to 0 degrees
- moved SW2 29.1 mm to (151.9, 53.0), turned to 0 degrees
- moved J1 26.5 mm to (152.5, 61.1), turned to -90 degrees
- moved C10 25.3 mm to (155.7, 69.0), turned to 90 degrees
- moved C18 24.1 mm to (155.7, 53.1), turned to -90 degrees
- moved R2 23.7 mm to (155.9, 67.0), turned to 180 degrees
- moved R7 22.8 mm to (155.9, 55.1), turned to 180 degrees
- moved J2 20.0 mm to (160.2, 69.0), turned to 90 degrees
- moved AE1 19.4 mm to (183.8, 65.5), turned to -90 degrees
- moved C13 18.9 mm to (158.5, 55.9), turned to 90 degrees
- moved R6 18.4 mm to (158.5, 62.9), turned to 0 degrees
- moved R5 18.0 mm to (158.5, 59.9), turned to 0 degrees
- moved C1 16.8 mm to (178.9, 69.2), turned to 0 degrees
- moved L2 16.5 mm to (160.3, 55.9), turned to 90 degrees
- moved C21 15.7 mm to (181.9, 63.1), turned to -90 degrees
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Other:
- board size 20 x 40.8 mm -> 40.8 x 20 mm
