File: PCB/esp.kicad_pcb (KiCad board)
At the start: 4 copper layers, 40.8 x 20 mm, 45 parts, among them J1 USB_C_Receptacle_USB2.0_14P, J2 Conn_01x04_Pin, SW1 RESET, SW2 BOOT, U1 ESP32-C3, U2 W25Q128JVP, U3 USBLC6-2P6, U4 MS5611-01BA, U5 SPX3819M5-L-3-3, U6 SHTC3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

Commit message: pushing before redoing everything
Parts:
- moved C9 0.53 mm to (171.3, 64.1)
Routing:
- net GND: track 40.0 -> 40.9 mm
Changed lines of the file:
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@@
 	(footprint "Capacitor_SMD:C_0402_1005Metric"
 		(layer "F.Cu")
-		(at 171.85 64.05 180)
+		(at 171.32 64.1 180)
 		(descr "Capacitor SMD 0402 (1005 Metric), square (rectangular) end terminal, IPC-7351 nominal, (Body size source: IPC-SM-782 page 76, https://www.pcb-3d.com/wordpress/wp-content/uploads/ipc-sm-782a_amendment_1_and_2.pdf), generated with kicad-footprint-generator")
 		(tags "capacitor")
@@
 	)
 	(segment
+		(start 170.6 64.1)
+		(end 170.1 63.6)
+		(width 0.2)
+		(layer "F.Cu")
+		(net 1)
+	)
+	(segment
+		(start 170.84 64.1)
+		(end 170.6 64.1)
+		(width 0.2)
+		(layer "F.Cu")
+		(net 1)
+	)
+	(segment
 		(start 172.025 69.2)
 		(end 171.7 68.875)
@@
 	)
 	(segment
+		(start 171.85 63.3)
+		(end 171.85 64.05)
+		(width 0.2)
+		(layer "F.Cu")
+		(net 4)
+	)
+	(segment
 		(start 168.5 56.4)
 		(end 167.25 55.15)
@@
 	)
 	(segment
-		(start 172.06 63.3)
-		(end 172.33 63.57)
-		(width 0.2)
-		(layer "F.Cu")
-		(net 4)
-	)
-	(segment
-		(start 172.33 63.57)
-		(end 172.33 64.05)
-		(width 0.2)
-		(layer "F.Cu")
-		(net 4)
-	)
-	(segment
 		(start 170.3 58.475)
 		(end 169.5 57.675)
@@
 		(layer "F.Cu")
 		(net 4)
+	)
+	(segment
+		(start 171.85 64.05)
+		(end 171.8 64.1)
+		(width 0.2)
+		(layer "F.Cu")
+		(net 4)
