File: PCB/esp.kicad_pcb (KiCad board)
At the start: 4 copper layers, 40.8 x 20 mm, 45 parts, among them J1 USB_C_Receptacle_USB2.0_14P, J2 Conn_01x04_Pin, SW1 RESET, SW2 BOOT, U1 ESP32-C3, U2 W25Q128JVP, U3 USBLC6-2P6, U4 MS5611-01BA, U5 SPX3819M5-L-3-3, U6 SHTC3, Y2 Crystal_GND24

Commit message: SD
Parts:
- added .: LOGO, LOGO, F.Cu at (190.8, 62.8)
- added TP1: TestPoint, Connector_PinHeader_1.00mm:PinHeader_1x01_P1.00mm_Vertical, B.Cu at (172.2, 52.0)
- added TP3: TestPoint, Connector_PinHeader_1.00mm:PinHeader_1x01_P1.00mm_Vertical, B.Cu at (166.8, 52.0)
Routing:
- net SCL: track 9.37 -> 12.8 mm
- net SDA: track 6.72 -> 8.71 mm, vias 0 -> 1
Other:
- board text added: "Made by Souptik Samanta"
